Commit message: red color

File: src/homewhere/urdf/box_robot.small.xacro (robot description, xacro)
@@ -62,5 +62,10 @@
         </geometry>
         <origin xyz="0 0 0" rpy="1.57 0 0" />
-        <material name="grey" />
+        <xacro:if value="${name == 'front_right'}">
+          <material name="red" />
+        </xacro:if>
+        <xacro:unless value="${name == 'front_right'}">
+          <material name="grey" />
+        </xacro:unless>
       </visual>
       <collision>
@@ -85,5 +90,10 @@
         </geometry>
         <origin xyz="0 0 0" rpy="0 0 0" />
-        <material name="green" />
+        <xacro:if value="${name == 'front_right'}">
+          <material name="red" />
+        </xacro:if>
+        <xacro:unless value="${name == 'front_right'}">
+          <material name="green" />
+        </xacro:unless>
       </visual>
       <inertial>

File: src/homewhere/urdf/color.gazebo.xacro (robot description, xacro)
@@ -21,5 +21,5 @@
   </gazebo>
   <gazebo reference="wheel_front_right">
-    <material>Gazebo/Grey </material>
+    <material>Gazebo/Red </material>
   </gazebo>
   <gazebo reference="wheel_rear_left">

Commit message: params

File: src/homewhere/urdf/box_robot.small.xacro (robot description, xacro)
@@ -112,5 +112,5 @@
       <origin xyz="${x} ${y} -0.1" rpy="0 0 0" />
       <axis xyz="0 0 1" />
-      <limit lower="${-3 * pi/2}" upper="${3 * pi/2}" effort="1000.0" velocity="0.1" />
+      <limit lower="${-pi/2}" upper="${pi/2}" effort="1000.0" velocity="0.1" />
     </joint>
     <!-- z = -leg/2 -->

Commit message: params

File: src/homewhere/urdf/box_robot.small.xacro (robot description, xacro)
@@ -112,5 +112,5 @@
       <origin xyz="${x} ${y} -0.1" rpy="0 0 0" />
       <axis xyz="0 0 1" />
-      <limit lower="${-pi/2}" upper="${pi/2}" effort="1000.0" velocity="0.1" />
+      <limit lower="${-3 * pi/2}" upper="${3 * pi/2}" effort="1000.0" velocity="0.1" />
     </joint>
     <!-- z = -leg/2 -->

Commit message: adjust value

File: src/homewhere/urdf/box_robot.small.xacro (robot description, xacro)
@@ -8,8 +8,7 @@
   <!-- ================== -->
   <xacro:property name="base_mass" value="20.0" />
-  <xacro:property name="base_size" value="0.25 0.25 0.1" />
+  <xacro:property name="base_size" value="0.25 0.25 0.25" />
   <xacro:property name="steer_mass" value="2.0" />
   <xacro:property name="steer_size" value="0.05 0.05 0.1" />
-  <!-- z of steer is 0.1 + radius of wheel -->
   <xacro:property name="wheel_mass" value="2.0" />
   <xacro:property name="wheel_radius" value="0.07" />
@@ -107,10 +106,20 @@
     </link>
     <!-- z = base_side/2 + leg/2 -->
-    <joint name="steer_${name}_joint" type="revolute">
+    <!-- <joint name="steer_${name}_joint" type="revolute">
       <parent link="body" />
       <child link="steer_${name}" />
       <origin xyz="${x} ${y} -0.1" rpy="0 0 0" />
       <axis xyz="0 0 1" />
-      <limit lower="${-3 * pi/2}" upper="${3 * pi/2}" effort="1000.0" velocity="0.1" />
+      <limit lower="${-pi/2}" upper="${pi/2}" effort="1000.0" velocity="0.1" />
+      <safety_controller soft_lower_limit="${-pi/2 * 0.9}" soft_upper_limit="${pi/2 * 0.9}" k_position="10.0" k_velocity="1000.0" />
+    </joint> -->
+    <!-- z = base_side/2 + leg/2 -->
+    <joint name="steer_${name}_joint" type="continuous">
+      <parent link="body" />
+      <child link="steer_${name}" />
+      <origin xyz="${x} ${y} -0.175" rpy="0 0 0" />
+      <axis xyz="0 0 1" />
+      <!-- <limit lower="${-pi/2}" upper="${pi/2}" effort="1000.0" velocity="0.1" />
+      <safety_controller soft_lower_limit="${-pi/2 * 0.9}" soft_upper_limit="${pi/2 * 0.9}" k_position="10.0" k_velocity="1000.0" /> -->
     </joint>
     <!-- z = -leg/2 -->
@@ -137,5 +146,5 @@
     <parent link="base_link" />
     <child link="base_scan" />
-    <origin xyz="0 0 0.1" rpy="0 0 0" />
+    <origin xyz="0 0 0.15" rpy="0 0 0" />
   </joint>
   <xacro:steering_wheel name="front_left" x="0.1" y="0.1" />

Commit message: init

File: src/homewhere/urdf/box_robot.small.xacro (robot description, xacro)
@@ -115,11 +115,12 @@
     </joint> -->
     <!-- z = base_side/2 + leg/2 -->
-    <joint name="steer_${name}_joint" type="continuous">
+    <joint name="steer_${name}_joint" type="revolute">
       <parent link="body" />
       <child link="steer_${name}" />
       <origin xyz="${x} ${y} -0.175" rpy="0 0 0" />
       <axis xyz="0 0 1" />
-      <!-- <limit lower="${-pi/2}" upper="${pi/2}" effort="1000.0" velocity="0.1" />
-      <safety_controller soft_lower_limit="${-pi/2 * 0.9}" soft_upper_limit="${pi/2 * 0.9}" k_position="10.0" k_velocity="1000.0" /> -->
+      <limit lower="${-pi/2}" upper="${pi/2}" effort="100.0" velocity="0.1" />
+      <dynamics damping="1.0" friction="0.5"/>
+      <!-- <safety_controller soft_lower_limit="${-pi/2 * 0.9}" soft_upper_limit="${pi/2 * 0.9}" k_position="10.0" k_velocity="1000.0" /> --> -->
     </joint>
     <!-- z = -leg/2 -->

Commit message: add: update

File: src/homewhere/urdf/box_robot.small.xacro (robot description, xacro)
@@ -8,7 +8,8 @@
   <!-- ================== -->
   <xacro:property name="base_mass" value="20.0" />
-  <xacro:property name="base_size" value="0.25 0.25 0.25" />
-  <xacro:property name="steer_mass" value="2.0" />
-  <xacro:property name="steer_size" value="0.05 0.05 0.1" />
+  <xacro:property name="base_size" value="0.5 0.5 0.5" />
+  <xacro:property name="steer_mass" value="2.5" />
+  <xacro:property name="steer_size" value="0.05 0.05 0.22" />
+  <!-- z of steer is 0.1 + radius of wheel -->
   <xacro:property name="wheel_mass" value="2.0" />
   <xacro:property name="wheel_radius" value="0.07" />
@@ -40,7 +41,7 @@
       <origin xyz="0 0 0" />
       <inertia
-        ixx="0.208" ixy="0.0" ixz="0.0"
-        iyy="0.208" iyz="0.0"
-        izz="0.208" />
+        ixx="0.833" ixy="0.0" ixz="0.0"
+        iyy="0.833" iyz="0.0"
+        izz="0.833" />
     </inertial>
   </link>
@@ -61,10 +62,5 @@
         </geometry>
         <origin xyz="0 0 0" rpy="1.57 0 0" />
-        <xacro:if value="${name == 'front_right'}">
-          <material name="red" />
-        </xacro:if>
-        <xacro:unless value="${name == 'front_right'}">
-          <material name="grey" />
-        </xacro:unless>
+        <material name="grey" />
       </visual>
       <collision>
@@ -89,11 +85,20 @@
         </geometry>
         <origin xyz="0 0 0" rpy="0 0 0" />
-        <xacro:if value="${name == 'front_right'}">
-          <material name="red" />
-        </xacro:if>
-        <xacro:unless value="${name == 'front_right'}">
-          <material name="green" />
-        </xacro:unless>
+        <material name="green" />
       </visual>
+      <!-- <collision>
+        <geometry>
+          <box size="${steer_size}" />
+        </geometry>
+        <origin xyz="0 0 0" rpy="0 0 0" />
+      </collision> -->
+      <!-- <inertial>
+        <mass value="${steer_mass}" />
+        <origin xyz="0 0 0" />
+        <inertia
+          ixx="0.0021" ixy="0.0" ixz="0.0"
+          iyy="0.0021" iyz="0.0"
+          izz="0.0008"/>
+      </inertial> -->
       <inertial>
         <mass value="${steer_mass}" />
@@ -106,20 +111,12 @@
     </link>
     <!-- z = base_side/2 + leg/2 -->
-    <!-- <joint name="steer_${name}_joint" type="revolute">
+    <joint name="steer_${name}_joint" type="revolute">
       <parent link="body" />
       <child link="steer_${name}" />
-      <origin xyz="${x} ${y} -0.1" rpy="0 0 0" />
+      <origin xyz="${x} ${y} -0.25" rpy="0 0 0" />
       <axis xyz="0 0 1" />
-      <limit lower="${-pi/2}" upper="${pi/2}" effort="1000.0" velocity="0.1" />
-      <safety_controller soft_lower_limit="${-pi/2 * 0.9}" soft_upper_limit="${pi/2 * 0.9}" k_position="10.0" k_velocity="1000.0" />
-    </joint> -->
-    <!-- z = base_side/2 + leg/2 -->
-    <joint name="steer_${name}_joint" type="continuous">
-      <parent link="body" />
-      <child link="steer_${name}" />
-      <origin xyz="${x} ${y} -0.175" rpy="0 0 0" />
-      <axis xyz="0 0 1" />
-      <!-- <limit lower="${-pi/2}" upper="${pi/2}" effort="1000.0" velocity="0.1" />
-      <safety_controller soft_lower_limit="${-pi/2 * 0.9}" soft_upper_limit="${pi/2 * 0.9}" k_position="10.0" k_velocity="1000.0" /> -->
+      <!-- Updated to positional control -->
+      <limit lower="${-3 * pi / 2}" upper="${3 * pi / 2}" effort="1000.0" velocity="314" />
+      <!-- Removed velocity control, since it's not needed for position -->
     </joint>
     <!-- z = -leg/2 -->
@@ -127,5 +124,5 @@
       <parent link="steer_${name}" />
       <child link="wheel_${name}" />
-      <origin xyz="0 0 -0.05" />
+      <origin xyz="0 0 -0.11" />
       <axis xyz="0 1 0" />
     </joint>
@@ -146,9 +143,9 @@
     <parent link="base_link" />
     <child link="base_scan" />
-    <origin xyz="0 0 0.15" rpy="0 0 0" />
+    <origin xyz="0 0 0.275" rpy="0 0 0" />
   </joint>
-  <xacro:steering_wheel name="front_left" x="0.1" y="0.1" />
-  <xacro:steering_wheel name="front_right" x="0.1" y="-0.1" />
-  <xacro:steering_wheel name="rear_left" x="-0.1" y="0.1" />
-  <xacro:steering_wheel name="rear_right" x="-0.1" y="-0.1" />
+  <xacro:steering_wheel name="front_left" x="0.2" y="0.2" />
+  <xacro:steering_wheel name="front_right" x="0.2" y="-0.2" />
+  <xacro:steering_wheel name="rear_left" x="-0.2" y="0.2" />
+  <xacro:steering_wheel name="rear_right" x="-0.2" y="-0.2" />
 </robot>

Commit message: add: servo_sim

File: src/homewhere/urdf/box_robot.small.xacro (robot description, xacro)
@@ -8,8 +8,7 @@
   <!-- ================== -->
   <xacro:property name="base_mass" value="20.0" />
-  <xacro:property name="base_size" value="0.5 0.5 0.5" />
-  <xacro:property name="steer_mass" value="2.5" />
-  <xacro:property name="steer_size" value="0.05 0.05 0.22" />
-  <!-- z of steer is 0.1 + radius of wheel -->
+  <xacro:property name="base_size" value="0.25 0.25 0.25" />
+  <xacro:property name="steer_mass" value="2.0" />
+  <xacro:property name="steer_size" value="0.05 0.05 0.1" />
   <xacro:property name="wheel_mass" value="2.0" />
   <xacro:property name="wheel_radius" value="0.07" />
@@ -41,7 +40,7 @@
       <origin xyz="0 0 0" />
       <inertia
-        ixx="0.833" ixy="0.0" ixz="0.0"
-        iyy="0.833" iyz="0.0"
-        izz="0.833" />
+        ixx="0.208" ixy="0.0" ixz="0.0"
+        iyy="0.208" iyz="0.0"
+        izz="0.208" />
     </inertial>
   </link>
@@ -62,5 +61,10 @@
         </geometry>
         <origin xyz="0 0 0" rpy="1.57 0 0" />
-        <material name="grey" />
+        <xacro:if value="${name == 'front_right'}">
+          <material name="red" />
+        </xacro:if>
+        <xacro:unless value="${name == 'front_right'}">
+          <material name="grey" />
+        </xacro:unless>
       </visual>
       <collision>
@@ -85,20 +89,11 @@
         </geometry>
         <origin xyz="0 0 0" rpy="0 0 0" />
-        <material name="green" />
+        <xacro:if value="${name == 'front_right'}">
+          <material name="red" />
+        </xacro:if>
+        <xacro:unless value="${name == 'front_right'}">
+          <material name="green" />
+        </xacro:unless>
       </visual>
-      <!-- <collision>
-        <geometry>
-          <box size="${steer_size}" />
-        </geometry>
-        <origin xyz="0 0 0" rpy="0 0 0" />
-      </collision> -->
-      <!-- <inertial>
-        <mass value="${steer_mass}" />
-        <origin xyz="0 0 0" />
-        <inertia
-          ixx="0.0021" ixy="0.0" ixz="0.0"
-          iyy="0.0021" iyz="0.0"
-          izz="0.0008"/>
-      </inertial> -->
       <inertial>
         <mass value="${steer_mass}" />
@@ -111,12 +106,20 @@
     </link>
     <!-- z = base_side/2 + leg/2 -->
-    <joint name="steer_${name}_joint" type="revolute">
+    <!-- <joint name="steer_${name}_joint" type="revolute">
       <parent link="body" />
       <child link="steer_${name}" />
-      <origin xyz="${x} ${y} -0.25" rpy="0 0 0" />
+      <origin xyz="${x} ${y} -0.1" rpy="0 0 0" />
       <axis xyz="0 0 1" />
-      <!-- Updated to positional control -->
-      <limit lower="${-3 * pi / 2}" upper="${3 * pi / 2}" effort="1000.0" velocity="314" />
-      <!-- Removed velocity control, since it's not needed for position -->
+      <limit lower="${-pi/2}" upper="${pi/2}" effort="1000.0" velocity="0.1" />
+      <safety_controller soft_lower_limit="${-pi/2 * 0.9}" soft_upper_limit="${pi/2 * 0.9}" k_position="10.0" k_velocity="1000.0" />
+    </joint> -->
+    <!-- z = base_side/2 + leg/2 -->
+    <joint name="steer_${name}_joint" type="continuous">
+      <parent link="body" />
+      <child link="steer_${name}" />
+      <origin xyz="${x} ${y} -0.175" rpy="0 0 0" />
+      <axis xyz="0 0 1" />
+      <!-- <limit lower="${-pi/2}" upper="${pi/2}" effort="1000.0" velocity="0.1" />
+      <safety_controller soft_lower_limit="${-pi/2 * 0.9}" soft_upper_limit="${pi/2 * 0.9}" k_position="10.0" k_velocity="1000.0" /> -->
     </joint>
     <!-- z = -leg/2 -->
@@ -124,5 +127,5 @@
       <parent link="steer_${name}" />
       <child link="wheel_${name}" />
-      <origin xyz="0 0 -0.11" />
+      <origin xyz="0 0 -0.05" />
       <axis xyz="0 1 0" />
     </joint>
@@ -143,9 +146,9 @@
     <parent link="base_link" />
     <child link="base_scan" />
-    <origin xyz="0 0 0.275" rpy="0 0 0" />
+    <origin xyz="0 0 0.15" rpy="0 0 0" />
   </joint>
-  <xacro:steering_wheel name="front_left" x="0.2" y="0.2" />
-  <xacro:steering_wheel name="front_right" x="0.2" y="-0.2" />
-  <xacro:steering_wheel name="rear_left" x="-0.2" y="0.2" />
-  <xacro:steering_wheel name="rear_right" x="-0.2" y="-0.2" />
+  <xacro:steering_wheel name="front_left" x="0.1" y="0.1" />
+  <xacro:steering_wheel name="front_right" x="0.1" y="-0.1" />
+  <xacro:steering_wheel name="rear_left" x="-0.1" y="0.1" />
+  <xacro:steering_wheel name="rear_right" x="-0.1" y="-0.1" />
 </robot>

Commit message: add ramp

File: src/homewhere/urdf/box_robot.small.xacro (robot description, xacro)
@@ -132,4 +132,20 @@
     </joint>
   </xacro:macro>
+    <!-- ============== -->
+    <!-- Imu link      -->
+    <!-- ============== -->
+    <link name="imu_link">
+      <visual>
+        <geometry>
+          <box size="0.02 0.02 0.02" />
+        </geometry>
+        <material name="red"/>
+      </visual>
+    </link>
+    <joint name="imu_joint" type="fixed">
+      <parent link="body"/>
+      <child link="imu_link"/>
+      <origin xyz="0 0 0.3" rpy="0 0 0"/>
+    </joint>
   <!-- ============== -->
   <!-- 3) Lidar       -->
@@ -147,5 +163,5 @@
     <parent link="base_link" />
     <child link="base_scan" />
-    <origin xyz="0 0 0.15" rpy="0 0 0" />
+    <origin xyz="0 0 0.15" rpy="0 -0.1 0" />
   </joint>
   <xacro:steering_wheel name="front_left" x="0.1" y="0.1" />

File: src/homewhere/urdf/box_robot.xacro (robot description, xacro)
@@ -126,4 +126,20 @@
     </joint>
   </xacro:macro>
+    <!-- ============== -->
+    <!-- Imu link      -->
+    <!-- ============== -->
+    <link name="imu_link">
+      <visual>
+        <geometry>
+          <box size="0.02 0.02 0.02" />
+        </geometry>
+        <material name="red"/>
+      </visual>
+    </link>
+    <joint name="imu_joint" type="fixed">
+      <parent link="body"/>
+      <child link="imu_link"/>
+      <origin xyz="0 0 0.3" rpy="0 0 0"/>
+    </joint>
   <!-- ============== -->
   <!-- 3) Lidar       -->
@@ -141,5 +157,5 @@
     <parent link="base_link" />
     <child link="base_scan" />
-    <origin xyz="0 0 0.275" rpy="0 0 0" />
+    <origin xyz="0 0 0.275" rpy="0 -0.05 0" />
   </joint>
   <xacro:steering_wheel name="front_left" x="0.2" y="0.2" />

File: src/homewhere/urdf/plugin.xacro (robot description, xacro)
@@ -6,5 +6,5 @@
     <gazebo reference="base_scan">
         <sensor type="ray" name="lidar_sensor">
-            <origin xyz="0 0 0.2" rpy="0 0 0" />
+            <origin xyz="0 0 0.2" rpy="0 -0.1 0" />
             <visualize>true</visualize>
             <update_rate>60</update_rate>
@@ -35,3 +35,23 @@
         </sensor>
     </gazebo>
+    <gazebo reference="imu_link">
+        <gravity>true</gravity>
+        <sensor name="imu_sensor" type="imu">
+        <always_on>true</always_on>
+        <update_rate>100</update_rate>
+        <visualize>true</visualize>
+        <topic>__default_topic__</topic>
+        <plugin filename="libgazebo_ros_imu_sensor.so" name="imu_plugin">
+            <topicName>imu</topicName>
+            <bodyName>imu_link</bodyName>
+            <updateRateHZ>10.0</updateRateHZ>
+            <gaussianNoise>0.0</gaussianNoise>
+            <xyzOffset>0 0 0</xyzOffset>
+            <rpyOffset>0 0 0</rpyOffset>
+            <frameName>imu_link</frameName>
+            <initialOrientationAsReference>false</initialOrientationAsReference>
+        </plugin>
+        <pose>0 0 0 0 0 0</pose>
+        </sensor>
+    </gazebo>
 </robot>

Commit message: fix

File: src/homewhere/urdf/box_robot.small.xacro (robot description, xacro)
@@ -115,11 +115,11 @@
     </joint> -->
     <!-- z = base_side/2 + leg/2 -->
-    <joint name="steer_${name}_joint" type="revolute">
+    <joint name="steer_${name}_joint" type="continuous">
       <parent link="body" />
       <child link="steer_${name}" />
       <origin xyz="${x} ${y} -0.175" rpy="0 0 0" />
       <axis xyz="0 0 1" />
-      <limit lower="${-pi/2}" upper="${pi/2}" effort="100.0" velocity="0.1" />
-      <dynamics damping="1.0" friction="0.5"/>
+      <!-- <limit lower="${-pi/2}" upper="${pi/2}" effort="100.0" velocity="0.1" />
+      <dynamics damping="1.0" friction="0.5"/> -->
       <!-- <safety_controller soft_lower_limit="${-pi/2 * 0.9}" soft_upper_limit="${pi/2 * 0.9}" k_position="10.0" k_velocity="1000.0" /> --> -->
     </joint>
