Commit message: multimap navigation

File: src/homewhere/urdf/plugin.xacro (robot description, xacro)
@@ -6,5 +6,5 @@
     <gazebo reference="base_scan">
         <sensor type="ray" name="lidar_sensor">
-            <origin xyz="0 0 0.2" rpy="0 0 0" />
+            <origin xyz="0 0 0.5" rpy="0 0 0" />
             <visualize>true</visualize>
             <update_rate>60</update_rate>
