Commit message: urdf

File: src/homewhere/urdf/box_robot.xacro (robot description, xacro)
@@ -1,25 +1,34 @@
 <?xml version="1.0"?>
-<robot name="rocker_bogie" xmlns:xacro="http://www.ros.org/wiki/xacro">
-  <!-- <xacro:include filename="$(find homewhere)/urdf/color.xacro" /> -->
+<robot name="box_robot" xmlns:xacro="http://www.ros.org/wiki/xacro">
+  <xacro:include filename="$(find homewhere)/urdf/color.xacro" />
+  <xacro:include filename="$(find homewhere)/urdf/color.gazebo.xacro" />
+  <xacro:include filename="$(find homewhere)/urdf/plugin.xacro" />
   <!-- ================== -->
-  <!-- 1) Base Link      -->
+  <!-- 0) Properties      -->
+  <!-- ================== -->
+  <xacro:property name="base_mass" value="10.0" />
+  <xacro:property name="base_size" value="0.5 0.5 0.5" />
+  <xacro:property name="steer_mass" value="5.0" />
+  <xacro:property name="steer_size" value="0.05 0.05 0.1" />
+  <xacro:property name="wheel_mass" value="4.0" />
+  <xacro:property name="wheel_radius" value="0.07" />
+  <xacro:property name="wheel_length" value="0.04" />
+  <!-- ================== -->
+  <!-- 1) Base Link       -->
   <!-- ================== -->
   <link name="base_link">
     <visual>
       <geometry>
-        <box size="0.5 0.5 0.5" />
+        <box size="${base_size}" />
       </geometry>
-      <material name="orange">
-        <color rgba="1.0 0.423529 0.0392157 1.0" />
-        <!-- <color rgba="${255/255} ${108/255} ${10/255} 1.0" /> -->
-      </material>
+      <material name="orange"/>
     </visual>
     <collision>
       <geometry>
-        <box size="0.5 0.5 0.5" />
+        <box size="${base_size}" />
       </geometry>
     </collision>
     <inertial>
-      <mass value="10" />
+      <mass value="${base_mass}" />
       <origin xyz="0 0 0" />
       <inertia ixx="0.1" ixy="0" ixz="0" iyy="0.1" iyz="0" izz="0.1" />
@@ -27,26 +36,42 @@
   </link>
   <!-- ============== -->
-  <!-- 2) Wheel      -->
+  <!-- 2) Wheel       -->
   <!-- ============== -->
-  <xacro:macro name="steering_joint" params="name x y">
+  <xacro:macro name="steering_wheel" params="name x y">
     <link name="steer_${name}">
       <visual>
         <geometry>
-          <box size="0.05 0.05 0.1" />
+          <box size="${steer_size}" />
         </geometry>
-        <material name="blue">
-          <color rgba="0 0 1 1" />
-        </material>
+        <material name="green"/>
       </visual>
+      <!-- <collision>
+        <geometry>
+          <box size="${steer_size}" />
+        </geometry>
+      </collision> -->
+      <inertial>
+        <mass value="${steer_mass}" />
+        <origin xyz="0 0 0" />
+        <inertia ixx="0.1" ixy="0" ixz="0" iyy="0.1" iyz="0" izz="0.1" />
+      </inertial>
     </link>
     <link name="wheel_${name}">
       <visual>
         <geometry>
-          <cylinder length="0.05" radius="0.05" />
+          <cylinder length="0.04" radius="0.07" />
         </geometry>
-        <material name="black">
-          <color rgba="0 0 0 1" />
-        </material>
+        <material name="black"/>
       </visual>
+      <collision>
+        <geometry>
+          <cylinder length="${wheel_length}" radius="${wheel_radius}" />
+        </geometry>
+      </collision>
+      <inertial>
+        <mass value="${wheel_mass}" />
+        <origin xyz="0 0 0" />
+        <inertia ixx="0.0005" ixy="0" ixz="0" iyy="0.0005" iyz="0" izz="0.001" />
+      </inertial>
     </link>
     <joint name="steer_${name}_joint" type="revolute">
@@ -55,17 +80,17 @@
       <origin xyz="${x} ${y} -0.3" rpy="0 0 0" />
       <axis xyz="0 0 1" />
-      <limit lower="-0.785" upper="0.785" effort="5.0" velocity="1.0" />
+      <limit lower="-0.785" upper="0.785" effort="10.0" velocity="2.0" />
     </joint>
-    <joint name="wheel_${name}_joint" type="revolute">
+    <joint name="wheel_${name}_joint" type="continuous">
       <parent link="steer_${name}" />
       <child link="wheel_${name}" />
       <origin xyz="0 0 -0.05" rpy="0 1.5708 0" />
       <axis xyz="0 0 1" />
-      <limit lower="-0.785" upper="0.785"/>
+      <!-- <limit lower="-0.785" upper="0.785" effort="10.0" velocity="2.0" /> -->
     </joint>
   </xacro:macro>
-  <xacro:steering_joint name="front_left" x="-0.2" y="0.2" />
-  <xacro:steering_joint name="front_right" x="0.2" y="0.2" />
-  <xacro:steering_joint name="rear_left" x="-0.2" y="-0.2" />
-  <xacro:steering_joint name="rear_right" x="0.2" y="-0.2" />
+  <xacro:steering_wheel name="front_left"   x="-0.2"  y="0.2" />
+  <xacro:steering_wheel name="front_right"  x="0.2"   y="0.2" />
+  <xacro:steering_wheel name="rear_left"    x="-0.2"  y="-0.2" />
+  <xacro:steering_wheel name="rear_right"   x="0.2"   y="-0.2" />
 </robot>

Commit message: inertia

File: src/homewhere/urdf/box_robot.xacro (robot description, xacro)
@@ -7,8 +7,9 @@
   <!-- 0) Properties      -->
   <!-- ================== -->
-  <xacro:property name="base_mass" value="10.0" />
+  <xacro:property name="base_mass" value="20.0" />
   <xacro:property name="base_size" value="0.5 0.5 0.5" />
-  <xacro:property name="steer_mass" value="5.0" />
-  <xacro:property name="steer_size" value="0.05 0.05 0.1" />
+  <xacro:property name="steer_mass" value="1.0" />
+  <xacro:property name="steer_size" value="0.05 0.05 0.22" />
+  <!-- z of steer is 0.1 + radius of wheel -->
   <xacro:property name="wheel_mass" value="4.0" />
   <xacro:property name="wheel_radius" value="0.07" />
@@ -32,5 +33,8 @@
       <mass value="${base_mass}" />
       <origin xyz="0 0 0" />
-      <inertia ixx="0.1" ixy="0" ixz="0" iyy="0.1" iyz="0" izz="0.1" />
+      <inertia
+        ixx="0.833" ixy="0.0" ixz="0.0"
+        iyy="0.833" iyz="0.0"
+        izz="0.833"/>
     </inertial>
   </link>
@@ -39,4 +43,28 @@
   <!-- ============== -->
   <xacro:macro name="steering_wheel" params="name x y">
+      <!-- roll = 1.57 to rotate the wheel upright-->
+    <link name="wheel_${name}">
+      <visual>
+        <geometry>
+          <cylinder length="${wheel_length}" radius="${wheel_radius}" />
+        </geometry>
+        <origin xyz="0 0 0" rpy="1.57 0 0" />
+        <material name="grey"/>
+      </visual>
+      <collision>
+        <geometry>
+          <cylinder length="${wheel_length}" radius="${wheel_radius}" />
+        </geometry>
+        <origin xyz="0 0 0" rpy="1.57 0 0" />
+      </collision>
+      <inertial>
+        <mass value="${wheel_mass}" />
+        <origin xyz="0 0 0"/>
+        <inertia
+          ixx="0.0054" ixy="0.0" ixz="0.0"
+          iyy="0.0098" iyz="0.0"
+          izz="0.0054"/>
+      </inertial>
+    </link>
     <link name="steer_${name}">
       <visual>
@@ -51,46 +79,41 @@
         </geometry>
       </collision> -->
+      <!-- <inertial>
+        <mass value="${steer_mass}" />
+        <origin xyz="0 0 0" />
+        <inertia
+          ixx="0.0021" ixy="0.0" ixz="0.0"
+          iyy="0.0021" iyz="0.0"
+          izz="0.0008"/>
+      </inertial> -->
       <inertial>
         <mass value="${steer_mass}" />
         <origin xyz="0 0 0" />
-        <inertia ixx="0.1" ixy="0" ixz="0" iyy="0.1" iyz="0" izz="0.1" />
+        <inertia
+          ixx="0" ixy="0" ixz="0"
+          iyy="0" iyz="0"
+          izz="0"/>
       </inertial>
     </link>
-    <link name="wheel_${name}">
-      <visual>
-        <geometry>
-          <cylinder length="0.04" radius="0.07" />
-        </geometry>
-        <material name="black"/>
-      </visual>
-      <collision>
-        <geometry>
-          <cylinder length="${wheel_length}" radius="${wheel_radius}" />
-        </geometry>
-      </collision>
-      <inertial>
-        <mass value="${wheel_mass}" />
-        <origin xyz="0 0 0" />
-        <inertia ixx="0.0005" ixy="0" ixz="0" iyy="0.0005" iyz="0" izz="0.001" />
-      </inertial>
-    </link>
+    <!-- z = base_side/2 + d_to_wheel = 0.5/2 + 0.04 -->
     <joint name="steer_${name}_joint" type="revolute">
       <parent link="base_link" />
       <child link="steer_${name}" />
-      <origin xyz="${x} ${y} -0.3" rpy="0 0 0" />
+      <origin xyz="${x} ${y} -0.25" rpy="0 0 0" />
       <axis xyz="0 0 1" />
-      <limit lower="-0.785" upper="0.785" effort="10.0" velocity="2.0" />
+      <limit lower="-0.785" upper="0.785" effort="10.0" velocity="0.1" />
     </joint>
+    <!-- z = -wheel_radius so the edge is at the center of the wheel -->
     <joint name="wheel_${name}_joint" type="continuous">
       <parent link="steer_${name}" />
       <child link="wheel_${name}" />
-      <origin xyz="0 0 -0.05" rpy="0 1.5708 0" />
-      <axis xyz="0 0 1" />
+      <origin xyz="0 0 -0.11"/>
+      <axis xyz="0 1 0" />
       <!-- <limit lower="-0.785" upper="0.785" effort="10.0" velocity="2.0" /> -->
     </joint>
   </xacro:macro>
-  <xacro:steering_wheel name="front_left"   x="-0.2"  y="0.2" />
-  <xacro:steering_wheel name="front_right"  x="0.2"   y="0.2" />
-  <xacro:steering_wheel name="rear_left"    x="-0.2"  y="-0.2" />
-  <xacro:steering_wheel name="rear_right"   x="0.2"   y="-0.2" />
+  <xacro:steering_wheel name="front_left"   x="0.2"  y="0.2" />
+  <xacro:steering_wheel name="front_right"  x="0.2"   y="-0.2" />
+  <xacro:steering_wheel name="rear_left"    x="-0.2"  y="0.2" />
+  <xacro:steering_wheel name="rear_right"   x="-0.2"   y="-0.2" />
 </robot>

Commit message: urdf

File: src/homewhere/urdf/box_robot.xacro (robot description, xacro)
@@ -9,8 +9,8 @@
   <xacro:property name="base_mass" value="20.0" />
   <xacro:property name="base_size" value="0.5 0.5 0.5" />
-  <xacro:property name="steer_mass" value="1.0" />
+  <xacro:property name="steer_mass" value="2.5" />
   <xacro:property name="steer_size" value="0.05 0.05 0.22" />
   <!-- z of steer is 0.1 + radius of wheel -->
-  <xacro:property name="wheel_mass" value="4.0" />
+  <xacro:property name="wheel_mass" value="2.0" />
   <xacro:property name="wheel_radius" value="0.07" />
   <xacro:property name="wheel_length" value="0.04" />
@@ -62,7 +62,7 @@
         <origin xyz="0 0 0"/>
         <inertia
-          ixx="0.0054" ixy="0.0" ixz="0.0"
-          iyy="0.0098" iyz="0.0"
-          izz="0.0054"/>
+          ixx="0.0027" ixy="0.0" ixz="0.0"
+          iyy="0.0049" iyz="0.0"
+          izz="0.0027"/>
       </inertial>
     </link>
@@ -102,5 +102,5 @@
       <origin xyz="${x} ${y} -0.25" rpy="0 0 0" />
       <axis xyz="0 0 1" />
-      <limit lower="-0.785" upper="0.785" effort="10.0" velocity="0.1" />
+      <limit lower="${-pi/2}" upper="${pi/2}" effort="1000.0" velocity="0.1" />
     </joint>
     <!-- z = -wheel_radius so the edge is at the center of the wheel -->
@@ -110,7 +110,23 @@
       <origin xyz="0 0 -0.11"/>
       <axis xyz="0 1 0" />
-      <!-- <limit lower="-0.785" upper="0.785" effort="10.0" velocity="2.0" /> -->
     </joint>
   </xacro:macro>
+  <!-- ============== -->
+  <!-- 3) Lidar       -->
+  <!-- ============== -->
+  <link name="base_scan">
+    <visual>
+      <!-- <origin xyz="0 0 0" rpy="0 0 0" /> -->
+      <geometry>
+        <cylinder length="0.05" radius="0.02" />
+      </geometry>
+      <material name="red"/>
+    </visual>
+  </link>
+  <joint name="scan_joint" type="fixed">
+    <parent link="base_link" />
+    <child link="base_scan" />
+    <origin xyz="0 0 0.275" rpy="0 0 0" />
+  </joint>
   <xacro:steering_wheel name="front_left"   x="0.2"  y="0.2" />
   <xacro:steering_wheel name="front_right"  x="0.2"   y="-0.2" />

File: src/homewhere/urdf/color.gazebo.xacro (robot description, xacro)
@@ -29,3 +29,6 @@
     <material>Gazebo/Grey </material>
   </gazebo>
+  <gazebo reference="base_scan">
+    <material>Gazebo/Red </material>
+  </gazebo>
 </robot>

File: src/homewhere/urdf/plugin.xacro (robot description, xacro)
@@ -2,5 +2,36 @@
 <robot name="plugin" xmlns:xacro="http://www.ros.org/wiki/xacro">
     <gazebo>
-        <plugin name="control_plugin" filename="libcontrol_plugin.so"/>
+        <plugin name="control_plugin" filename="libcontrol_plugin.so" />
+    </gazebo>
+    <gazebo reference="base_scan">
+        <sensor type="ray" name="lidar_sensor">
+            <origin xyz="0 0 0.2" rpy="0 0 0" />
+            <visualize>true</visualize>
+            <update_rate>60</update_rate>
+            <ray>
+                <scan>
+                    <horizontal>
+                        <samples>360</samples>
+                        <resolution>1</resolution>
+                        <min_angle>0</min_angle> <!-- -90 degrees -->
+                        <max_angle>6.28319</max_angle>  <!-- +90 degrees -->
+                    </horizontal>
+                </scan>
+                <range>
+                    <min>0.15</min> <!-- Min detection distance -->
+                    <max>3.5</max> <!-- Max detection distance -->
+                    <resolution>0.01</resolution>
+                </range>
+                <noise>
+                    <type>gaussian</type>
+                    <mean>0.0</mean>
+                    <stddev>0.01</stddev>
+                </noise>
+            </ray>
+            <plugin name="gazebo_ros_laser" filename="libgazebo_ros_laser.so">
+                <topicName>scan</topicName>
+                <frameName>base_scan</frameName>
+            </plugin>
+        </sensor>
     </gazebo>
 </robot>

Commit message: update: NAV1

File: src/homewhere/urdf/box_robot.xacro (robot description, xacro)
@@ -15,13 +15,20 @@
   <xacro:property name="wheel_radius" value="0.07" />
   <xacro:property name="wheel_length" value="0.04" />
+  <link name="base_link"></link>
+  <link name="base_footprint" />
+  <joint name="base_joint" type="fixed">
+    <parent link="base_footprint" />
+    <child link="base_link" />
+    <origin xyz="0 0 0" rpy="0 0 0" />
+  </joint>
   <!-- ================== -->
   <!-- 1) Base Link       -->
   <!-- ================== -->
-  <link name="base_link">
+  <link name="body">
     <visual>
       <geometry>
         <box size="${base_size}" />
       </geometry>
-      <material name="orange"/>
+      <material name="orange" />
     </visual>
     <collision>
@@ -36,12 +43,17 @@
         ixx="0.833" ixy="0.0" ixz="0.0"
         iyy="0.833" iyz="0.0"
-        izz="0.833"/>
+        izz="0.833" />
     </inertial>
   </link>
+  <joint name="base_to_body" type="fixed">
+    <parent link="base_link" />
+    <child link="body" />
+    <origin xyz="0 0 0" />
+  </joint>
   <!-- ============== -->
   <!-- 2) Wheel       -->
   <!-- ============== -->
   <xacro:macro name="steering_wheel" params="name x y">
-      <!-- roll = 1.57 to rotate the wheel upright-->
+    <!-- roll = 1.57 to rotate the wheel upright-->
     <link name="wheel_${name}">
       <visual>
@@ -50,5 +62,5 @@
         </geometry>
         <origin xyz="0 0 0" rpy="1.57 0 0" />
-        <material name="grey"/>
+        <material name="grey" />
       </visual>
       <collision>
@@ -60,9 +72,9 @@
       <inertial>
         <mass value="${wheel_mass}" />
-        <origin xyz="0 0 0"/>
+        <origin xyz="0 0 0" />
         <inertia
           ixx="0.0027" ixy="0.0" ixz="0.0"
           iyy="0.0049" iyz="0.0"
-          izz="0.0027"/>
+          izz="0.0027" />
       </inertial>
     </link>
@@ -72,5 +84,6 @@
           <box size="${steer_size}" />
         </geometry>
-        <material name="green"/>
+        <origin xyz="0 0 0" rpy="0 0 0" />
+        <material name="green" />
       </visual>
       <!-- <collision>
@@ -78,4 +91,5 @@
           <box size="${steer_size}" />
         </geometry>
+        <origin xyz="0 0 0" rpy="0 0 0" />
       </collision> -->
       <!-- <inertial>
@@ -93,20 +107,20 @@
           ixx="0" ixy="0" ixz="0"
           iyy="0" iyz="0"
-          izz="0"/>
+          izz="0" />
       </inertial>
     </link>
-    <!-- z = base_side/2 + d_to_wheel = 0.5/2 + 0.04 -->
+    <!-- z = base_side/2 + leg/2 -->
     <joint name="steer_${name}_joint" type="revolute">
-      <parent link="base_link" />
+      <parent link="body" />
       <child link="steer_${name}" />
       <origin xyz="${x} ${y} -0.25" rpy="0 0 0" />
       <axis xyz="0 0 1" />
-      <limit lower="${-pi/2}" upper="${pi/2}" effort="1000.0" velocity="0.1" />
+      <limit lower="${-3 * pi/2}" upper="${3 * pi/2}" effort="1000.0" velocity="0.1" />
     </joint>
-    <!-- z = -wheel_radius so the edge is at the center of the wheel -->
+    <!-- z = -leg/2 -->
     <joint name="wheel_${name}_joint" type="continuous">
       <parent link="steer_${name}" />
       <child link="wheel_${name}" />
-      <origin xyz="0 0 -0.11"/>
+      <origin xyz="0 0 -0.11" />
       <axis xyz="0 1 0" />
     </joint>
@@ -121,5 +135,5 @@
         <cylinder length="0.05" radius="0.02" />
       </geometry>
-      <material name="red"/>
+      <material name="red" />
     </visual>
   </link>
@@ -129,7 +143,7 @@
     <origin xyz="0 0 0.275" rpy="0 0 0" />
   </joint>
-  <xacro:steering_wheel name="front_left"   x="0.2"  y="0.2" />
-  <xacro:steering_wheel name="front_right"  x="0.2"   y="-0.2" />
-  <xacro:steering_wheel name="rear_left"    x="-0.2"  y="0.2" />
-  <xacro:steering_wheel name="rear_right"   x="-0.2"   y="-0.2" />
+  <xacro:steering_wheel name="front_left" x="0.2" y="0.2" />
+  <xacro:steering_wheel name="front_right" x="0.2" y="-0.2" />
+  <xacro:steering_wheel name="rear_left" x="-0.2" y="0.2" />
+  <xacro:steering_wheel name="rear_right" x="-0.2" y="-0.2" />
 </robot>

File: src/homewhere/urdf/color.gazebo.xacro (robot description, xacro)
@@ -2,5 +2,5 @@
 <robot name="color_gazebo" xmlns:xacro="http://www.ros.org/wiki/xacro">
   <!-- http://wiki.ros.org/simulator_gazebo/Tutorials/ListOfMaterials -->
-  <gazebo reference="base_link">
+  <gazebo reference="body">
     <material>Gazebo/Orange</material>
   </gazebo>

File: src/homewhere/urdf/plugin.xacro (robot description, xacro)
@@ -19,5 +19,5 @@
                 </scan>
                 <range>
-                    <min>0.15</min> <!-- Min detection distance -->
+                    <min>0.12</min> <!-- Min detection distance -->
                     <max>3.5</max> <!-- Max detection distance -->
                     <resolution>0.01</resolution>

Commit message: add: position control

File: src/homewhere/urdf/box_robot.xacro (robot description, xacro)
@@ -116,5 +116,7 @@
       <origin xyz="${x} ${y} -0.25" rpy="0 0 0" />
       <axis xyz="0 0 1" />
-      <limit lower="${-3 * pi/2}" upper="${3 * pi/2}" effort="1000.0" velocity="0.1" />
+      <!-- Updated to positional control -->
+      <limit lower="${-3 * pi / 2}" upper="${3 * pi / 2}" effort="1000.0" />
+      <!-- Removed velocity control, since it's not needed for position -->
     </joint>
     <!-- z = -leg/2 -->

Commit message: param

File: src/homewhere/urdf/box_robot.xacro (robot description, xacro)
@@ -111,10 +111,10 @@
     </link>
     <!-- z = base_side/2 + leg/2 -->
-    <joint name="steer_${name}_joint" type="revolute">
+    <joint name="steer_${name}_joint" type="continuous">
       <parent link="body" />
       <child link="steer_${name}" />
       <origin xyz="${x} ${y} -0.25" rpy="0 0 0" />
       <axis xyz="0 0 1" />
-      <limit lower="${-3 * pi/2}" upper="${3 * pi/2}" effort="1000.0" velocity="0.1" />
+      <!-- <limit lower="${-3 * pi/2}" upper="${3 * pi/2}" effort="1000.0" velocity="0.1" /> -->
     </joint>
     <!-- z = -leg/2 -->

Commit message: change small robot to big robot

File: src/homewhere/urdf/box_robot.xacro (robot description, xacro)
@@ -117,5 +117,5 @@
       <axis xyz="0 0 1" />
       <!-- Updated to positional control -->
-      <limit lower="${-3 * pi / 2}" upper="${3 * pi / 2}" effort="1000.0" />
+      <limit lower="${-3 * pi / 2}" upper="${3 * pi / 2}" effort="1000.0" velocity="1.0" />
       <!-- Removed velocity control, since it's not needed for position -->
     </joint>

Commit message: modify 17april

File: src/homewhere/urdf/box_robot.xacro (robot description, xacro)
@@ -157,5 +157,5 @@
     <parent link="base_link" />
     <child link="base_scan" />
-    <origin xyz="0 0 0.275" rpy="0 -0.05 0" />
+    <origin xyz="0 0 0.275" rpy="0 0.05 0" />
   </joint>
   <xacro:steering_wheel name="front_left" x="0.2" y="0.2" />

File: src/homewhere/urdf/plugin.xacro (robot description, xacro)
@@ -12,8 +12,8 @@
                 <scan>
                     <horizontal>
-                        <samples>360</samples>
+                        <samples>720</samples>
                         <resolution>1</resolution>
-                        <min_angle>0</min_angle> <!-- -90 degrees -->
-                        <max_angle>6.28319</max_angle>  <!-- +90 degrees -->
+                        <min_angle>-3.14159</min_angle> <!-- -90 degrees -->
+                        <max_angle>3.14159</max_angle>  <!-- +90 degrees -->
                     </horizontal>
                 </scan>

Commit message: imu plugin

File: src/homewhere/urdf/box_robot.xacro (robot description, xacro)
@@ -143,4 +143,14 @@
     <origin xyz="0 0 0.275" rpy="0 0 0" />
   </joint>
+  <!-- ============== -->
+  <!-- 4) Imu       -->
+  <!-- ============== -->
+  <link name="imu_link">
+  </link>
+  <joint name="imu_joint" type="fixed">
+    <parent link="base_link" />
+    <child link="imu_link" />
+    <origin xyz="0 0 0" rpy="0 0 0" />
+  </joint>
   <xacro:steering_wheel name="front_left" x="0.2" y="0.2" />
   <xacro:steering_wheel name="front_right" x="0.2" y="-0.2" />

File: src/homewhere/urdf/plugin.xacro (robot description, xacro)
@@ -35,3 +35,23 @@
         </sensor>
     </gazebo>
+    <gazebo reference="imu_link">
+        <gravity>true</gravity>
+        <sensor name="imu_sensor" type="imu">
+            <always_on>true</always_on>
+            <update_rate>100</update_rate>
+            <visualize>true</visualize>
+            <topic>__default_topic__</topic>
+            <plugin filename="libgazebo_ros_imu_sensor.so" name="imu_plugin">
+                <topicName>imu</topicName>
+                <bodyName>imu_link</bodyName>
+                <updateRateHZ>10.0</updateRateHZ>
+                <gaussianNoise>0.0</gaussianNoise>
+                <xyzOffset>0 0 0</xyzOffset>
+                <rpyOffset>0 0 0</rpyOffset>
+                <frameName>imu_link</frameName>
+                <initialOrientationAsReference>false</initialOrientationAsReference>
+            </plugin>
+            <pose>0 0 0 0 0 0</pose>
+        </sensor>
+    </gazebo>
 </robot>
